File: Hardware/LAB-PLR1010/CAD/LAB-PLR1010.sch (EAGLE design)
At the start: 8 parts, among them IC1 LT1963AEQ, U1 AD5270BRMZ-50

Commit message: 1) Updates to the LAB-PLR1010
Parts:
- removed IC1: LT1963AEQ, linear-technology:LT1963AEQ
- removed R1: 1R0, rcl:R-US_R2512
- added U2: LT3080EMS8EPBF, LAB-PLR1010:LT3080EMS8EPBF
Connections:
- removed net N$9: IC1.OUT, R1.2
- new net VOUT: SV1.3, U2.EP, U2.OUT, U2.OUT_2, U2.OUT_3
- net N$8: now also U2.SET; no longer IC1.SENSE
- net PE: no longer IC1.GND, IC1.GND@1, R1.1, SV1.3
- net VDDIO: now also U2.VCONTROL
- net VDDLDO: now also U2.IN, U2.IN_2; no longer IC1.!SHDN, IC1.IN
Changed lines of the file:
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@@
 <?xml version="1.0" encoding="utf-8"?>
 <!DOCTYPE eagle SYSTEM "eagle.dtd">
-<eagle version="6.5.0">
+<eagle version="6.6.0">
 <drawing>
 <settings>
@@
 <part name="U1" library="Analog Devices_By_element14_Batch_1" deviceset="AD5270BRMZ-50" device=""/>
 <part name="FRAME1" library="frames" deviceset="FRAME_A_L" device=""/>
-<part name="IC1" library="linear-technology" deviceset="LT1963AEQ*" device=""/>
 <part name="SV1" library="LAB304" deviceset="MA04-1" device=""/>
 <part name="SV2" library="LAB304" deviceset="MA04-1" device=""/>
-<part name="R1" library="rcl" deviceset="R-US_" device="R2512" value="1R0"/>
-<part name="PE1" library="supply1" deviceset="PE" device=""/>
-<part name="PE2" library="supply1" deviceset="PE" device=""/>
 <part name="PE3" library="supply1" deviceset="PE" device=""/>
 <part name="PE4" library="supply1" deviceset="PE" device=""/>
@@
 <part name="C3" library="SparkFun-Capacitors" deviceset="1NF/1000PF-50V-10%(0603)" device="" value="10uF"/>
 <part name="PE5" library="supply1" deviceset="PE" device=""/>
+<part name="U2" library="LAB-PLR1010" deviceset="LT3080EMS8EPBF" device=""/>
 </parts>
 <sheets>
@@
 <instance part="FRAME1" gate="G$1" x="0" y="0"/>
 <instance part="FRAME1" gate="G$2" x="172.72" y="0"/>
-<instance part="IC1" gate="A" x="208.28" y="114.3"/>
 <instance part="SV1" gate="1" x="43.18" y="116.84" rot="MR180"/>
 <instance part="SV2" gate="1" x="43.18" y="99.06" rot="MR180"/>
-<instance part="R1" gate="G$1" x="246.38" y="104.14" rot="R90"/>
-<instance part="PE1" gate="M" x="210.82" y="99.06"/>
-<instance part="PE2" gate="M" x="246.38" y="91.44"/>
 <instance part="PE3" gate="M" x="119.38" y="91.44"/>
 <instance part="PE4" gate="M" x="170.18" y="109.22"/>
@@
 <instance part="C3" gate="G$1" x="93.98" y="101.6" rot="MR0"/>
 <instance part="PE5" gate="M" x="71.12" y="114.3" rot="MR0"/>
+<instance part="U2" gate="A" x="215.9" y="109.22"/>
 </instances>
 <busses>
@@
 <net name="N$8" class="0">
 <segment>
-<pinref part="IC1" gate="A" pin="SENSE"/>
-<wire x1="223.52" y1="114.3" x2="220.98" y2="114.3" width="0.1524" layer="91"/>
 <pinref part="U1" gate="A" pin="W"/>
 <wire x1="160.02" y1="109.22" x2="162.56" y2="109.22" width="0.1524" layer="91"/>
-<wire x1="162.56" y1="109.22" x2="162.56" y2="93.98" width="0.1524" layer="91"/>
-<wire x1="162.56" y1="93.98" x2="223.52" y2="93.98" width="0.1524" layer="91"/>
-<wire x1="223.52" y1="93.98" x2="223.52" y2="114.3" width="0.1524" layer="91"/>
-</segment>
-</net>
-<net name="N$9" class="0">
-<segment>
-<pinref part="IC1" gate="A" pin="OUT"/>
-<pinref part="R1" gate="G$1" pin="2"/>
-<wire x1="220.98" y1="116.84" x2="246.38" y2="116.84" width="0.1524" layer="91"/>
-<wire x1="246.38" y1="116.84" x2="246.38" y2="109.22" width="0.1524" layer="91"/>
+<wire x1="162.56" y1="109.22" x2="162.56" y2="101.6" width="0.1524" layer="91"/>
+<pinref part="U2" gate="A" pin="SET"/>
+<wire x1="198.12" y1="101.6" x2="162.56" y2="101.6" width="0.1524" layer="91"/>
 </segment>
 </net>
 <net name="PE" class="0">
-<segment>
-<pinref part="IC1" gate="A" pin="GND"/>
-<wire x1="208.28" y1="104.14" x2="208.28" y2="101.6" width="0.1524" layer="91"/>
-<wire x1="208.28" y1="101.6" x2="210.82" y2="101.6" width="0.1524" layer="91"/>
-<pinref part="IC1" gate="A" pin="GND@1"/>
-<wire x1="210.82" y1="101.6" x2="210.82" y2="104.14" width="0.1524" layer="91"/>
-<pinref part="PE1" gate="M" pin="PE"/>
-<junction x="210.82" y="101.6"/>
-</segment>
-<segment>
-<pinref part="R1" gate="G$1" pin="1"/>
-<pinref part="PE2" gate="M" pin="PE"/>
-<wire x1="246.38" y1="93.98" x2="246.38" y2="99.06" width="0.1524" layer="91"/>
-</segment>
 <segment>
 <pinref part="U1" gate="A" pin="GND"/>
@@
 <wire x1="50.8" y1="119.38" x2="71.12" y2="119.38" width="0.1524" layer="91"/>
 <wire x1="71.12" y1="119.38" x2="71.12" y2="116.84" width="0.1524" layer="91"/>
-<pinref part="SV1" gate="1" pin="3"/>
-<wire x1="71.12" y1="116.84" x2="50.8" y2="116.84" width="0.1524" layer="91"/>
-<junction x="71.12" y="116.84"/>
 </segment>
 </net>
@@
 <label x="63.5" y="104.14" size="1.778" layer="95" rot="MR0"/>
 </segment>
+<segment>
+<pinref part="U2" gate="A" pin="VCONTROL"/>
+<wire x1="198.12" y1="114.3" x2="180.34" y2="114.3" width="0.1524" layer="91"/>
+<label x="180.34" y="114.3" size="1.778" layer="95"/>
+</segment>
 </net>
 <net name="VDDLDO" class="0">
-<segment>
-<pinref part="IC1" gate="A" pin="IN"/>
-<wire x1="198.12" y1="116.84" x2="195.58" y2="116.84" width="0.1524" layer="91"/>
-<pinref part="IC1" gate="A" pin="!SHDN"/>
-<wire x1="198.12" y1="111.76" x2="195.58" y2="111.76" width="0.1524" layer="91"/>
-<wire x1="195.58" y1="111.76" x2="195.58" y2="116.84" width="0.1524" layer="91"/>
-<junction x="195.58" y="116.84"/>
-<wire x1="195.58" y1="116.84" x2="182.88" y2="116.84" width="0.1524" layer="91"/>
-<label x="182.88" y="116.84" size="1.778" layer="95"/>
-</segment>
 <segment>
 <wire x1="50.8" y1="121.92" x2="63.5" y2="121.92" width="0.1524" layer="91"/>
@@
 <label x="63.5" y="121.92" size="1.778" layer="95" rot="MR0"/>
 </segment>
+<segment>
+<wire x1="198.12" y1="109.22" x2="180.34" y2="109.22" width="0.1524" layer="91"/>
+<pinref part="U2" gate="A" pin="IN_2"/>
+<label x="180.34" y="109.22" size="1.778" layer="95"/>
+</segment>
+<segment>
+<wire x1="198.12" y1="106.68" x2="180.34" y2="106.68" width="0.1524" layer="91"/>
+<pinref part="U2" gate="A" pin="IN"/>
+<label x="180.34" y="106.68" size="1.778" layer="95"/>
+</segment>
 </net>
 <net name="#CS" class="0">
@@
 </segment>
 </net>
+<net name="VOUT" class="0">
+<segment>
+<pinref part="U2" gate="A" pin="EP"/>
+<wire x1="233.68" y1="114.3" x2="236.22" y2="114.3" width="0.1524" layer="91"/>
+<wire x1="236.22" y1="114.3" x2="236.22" y2="111.76" width="0.1524" layer="91"/>
+<pinref part="U2" gate="A" pin="OUT"/>
+<wire x1="236.22" y1="111.76" x2="236.22" y2="109.22" width="0.1524" layer="91"/>
+<wire x1="236.22" y1="109.22" x2="236.22" y2="106.68" width="0.1524" layer="91"/>
+<wire x1="236.22" y1="106.68" x2="233.68" y2="106.68" width="0.1524" layer="91"/>
+<pinref part="U2" gate="A" pin="OUT_3"/>
+<wire x1="233.68" y1="109.22" x2="236.22" y2="109.22" width="0.1524" layer="91"/>
+<junction x="236.22" y="109.22"/>
+<pinref part="U2" gate="A" pin="OUT_2"/>
+<wire x1="233.68" y1="111.76" x2="236.22" y2="111.76" width="0.1524" layer="91"/>
+<junction x="236.22" y="111.76"/>
+<wire x1="236.22" y1="114.3" x2="246.38" y2="114.3" width="0.1524" layer="91"/>
+<junction x="236.22" y="114.3"/>
+<label x="246.38" y="114.3" size="1.778" layer="95" rot="MR0"/>
+</segment>
+<segment>
+<pinref part="SV1" gate="1" pin="3"/>
+<wire x1="50.8" y1="116.84" x2="63.5" y2="116.84" width="0.1524" layer="91"/>
+<label x="63.5" y="116.84" size="1.778" layer="95" rot="MR0"/>
+</segment>
+</net>

Commit message: 1) Updates to the PLR1010 + datasheet and bills of materials
Parts:
- removed C3: 10uF, SparkFun-Capacitors:1NF/1000PF-50V-10%(0603)
- removed SV1, SV2: (no value), LAB304:MA04-1
- added J1: (no value), con-lstb:MA10-1W
- added J2, J3: 22-23-2021, My Library-adm:22-23-2021
- added U3: LT3080, LAB-PLR1010:LT3080
- C1: value 1uF -> 10uF
- U1: value AD5270BRMZ-50 -> DAC8562; device Analog Devices_By_element14_Batch_1:AD5270BRMZ-50 -> LAB-PLR1010:DAC8562
- U2: value LT3080EMS8EPBF -> LT3080; device LAB-PLR1010:LT3080EMS8EPBF -> LAB-PLR1010:LT3080
Connections:
- removed net #CS: SV2.4, U1.~SYNC
- removed net MISO: SV2.2, U1.SDO
- removed net N$1: C1.1, U1.EXT_CAP
- removed net N$8: U1.W, U2.SET
- removed net PE: C1.2, C2.2, C3.2, SV1.2, U1.A, U1.GND, U1.VSS
- removed net VOUT: SV1.3, U2.EP, U2.OUT, U2.OUT_2, U2.OUT_3
- new net !CLR: J1.3, U1.!CLR
- new net !CS: J1.7, U1.!CS
- new net !LDAC: J1.2, U1.!LDAC
- new net GND: C1.2, C2.2, J1.5, J2-2.S, J3-1.S, U1.GND
- new net N$2: U1.VA, U2.SET
- new net N$3: U1.VB, U3.SET
- new net VA: J1.1, J2-1.S, U2.OUT
- new net VB: J1.10, J3-2.S, U3.OUT
- net MCLK: now also J1.8; no longer SV1.4
- net MOSI: now also J1.9; no longer SV2.3
- net VDDIO: now also C1.1, J1.6, U1.AVDD, U2.VCNTRL, U3.VCNTRL; no longer C3.1, SV2.1, U1.VDD, U2.VCONTROL
- net VDDLDO: now also J1.4, U1.REFIN/OUT, U3.IN; no longer SV1.1, U2.IN_2
Other:
- moved on the sheet: C1, C2
