File: Hardware/LAB-PRIME/cad/LAB-PRIME.brd (EAGLE design)
At the start: 160 x 100 mm, 48 parts, among them IC1 MT48LC16M16A2, IC2 25AA080SN, IC3 MT29F8G08DAA, IC4 FT232RL, U1 STM32F429IGT, U13 MAX4376, U2 LTC1982ES6PBF, U3 DMG6968U-7, U4 TPS62240DDC, U50 MCP601R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

Commit message: 1) Adding the ADSM300F to the LAB304 library 2) Quick updates to the prime board -- spacing related, preliminary 3) Fixing some library pointers in the PPS330D project file
Parts:
- added U$1, U$2, U$3, U$4: LAB-ADSM300F, LAB304:LAB-ASDM300F
- added U$5, U$6, U$7, U$8: LAB-PPS330D, LAB304:LAB-PPS330D
- moved IC3 209.0 mm to (7.16, 55.1), turned to 90 degrees
- moved IC4 203.6 mm to (7.53, 36.4)
- moved X1 166.6 mm to (85.0, 10.0), flipped to the bottom
- moved IC1 114.0 mm to (8.11, 79.5)
- moved U1 37.6 mm to (50.0, 50.0), turned to 45 degrees
Connections:
- new net VIN: U$1.8, U$2.8, U$3.8, U$4.8
- net GND: now also U$1.4, U$1.6, U$2.4, U$2.6, U$3.4, U$3.6, U$4.4, U$4.6, U$5.4, U$6.4, U$7.4, U$8.4
- net V0: now also U$5.3, U$6.3, U$7.3, U$8.3
Other:
- board size 160 x 100 mm -> 100 x 100 mm
