File: Hardware/LAB-DEB429A/cad/LAB-DEB429.brd (EAGLE design)
At the start: 149.9 x 99.1 mm, 96 parts, among them J1 TSW-132-02-S-D, U1 LAB-ADSM300F, U10 SF-MICROSD, U11 25AA512, U12 LAB-PPS330D, U13 LAB-PPS330D, U14 LAB-PPS330D, U15 SI1143, U16 LAB-PPS330D, U17 25AA512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

Commit message: 1) Releasing first revision to MFG
Parts:
- removed U$2: UM232H, LAB304:UM232H
- added R10, R15, R16, R17, R18, R19: (no value), rcl:0204/7
- added U27: UM232H, LAB304:UM232H
- C10, C6, C7, C8, C9: value 10u -> 0.1u
- C14: value 47u -> 10u
- C15: value 0.22u -> 10u
- C16, C19, C20: value 0.1u -> 10u
- C21: value 0.1u -> 0.22u
- C22: value 0.1u -> 47u
- U11: value 25AA512 -> 25MPX
- U17: value 25AA512 -> SST26VF; device PEGMA:SO-08M -> LAB304:SO-08M
- moved C22 149.3 mm to (11.7, 4.37), turned to 270 degrees
- moved C12 126.3 mm to (75.6, 117.2), turned to 0 degrees
- moved C14 102.8 mm to (71.1, 88.3), turned to 90 degrees
- moved C7 99.6 mm to (16.5, 5.56), turned to 180 degrees
- moved C21 81.0 mm to (10.8, 10.5), turned to 90 degrees
- moved C9 78.8 mm to (5.08, 87.0), turned to 90 degrees
- moved C19 72.8 mm to (75.6, 106.4), turned to 0 degrees
- moved C8 70.7 mm to (70.2, 19.7), turned to 180 degrees
- moved C6 68.8 mm to (26.4, 62.2), turned to 0 degrees
- moved U7 58.9 mm to (75.6, 109.4)
- moved R12 58.0 mm to (69.5, 116.4), turned to 0 degrees
- moved R5 57.3 mm to (80.6, 112.7)
- moved R6 57.3 mm to (82.7, 112.7)
- moved C4 57.1 mm to (82.7, 109.4)
- moved R7 57.1 mm to (80.6, 109.4)
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- renumbered U$1 to U26, X1 to U25, X2 to J2
Connections:
- net FMC_A24 renamed LD3
- net FMC_A25 renamed LD4
- net LCD_B1 renamed LCD_B4
- net LCD_B9 renamed LCD_B7
- net MCU_SWK renamed MCU_SWC
- removed net !PLR_LDAC: U22.!LDAC, U23.!LDAC, U24.!LDAC
- removed net BOOT1: J2.30
- removed net FMC_NE1: J1.35
- removed net PV_DCHRG: J1.12
- removed net USB_OTG_FS_ID: J2.50
- new net FMC_D14: J2.53
- new net FMC_D15: J2.56
- new net N$176: R17.2, U22.CHB
- new net N$177: R19.2, U22.MCLK
- new net N$178: R16.2, U23.MCLK
- new net N$179: R15.2, U23.CHB
- new net N$180: R10.2, U24.MCLK
- new net N$181: R18.2, U24.CHB
- new net N$182: R13.1, R14.2, U21.5
- new net N$183: R11.1, R12.2, U21.3
- net !PLR0_CS: now also U22.!CLR; no longer U22.!CS
- net !PLR1_CS: now also U23.!CLR; no longer U23.!CS
- net !PLR2_CS: now also U24.!CLR; no longer U24.!CS
- net !PLR_CLR: now also J2.50, U22.!CS, U23.!CS, U24.!CS; no longer U22.!CLR, U23.!CLR, U24.!CLR
- net !USB_RST: now also J2.30, U27.!RST, U27.PU1; no longer U$2.!RST, U$2.PU1
- net !WF_RESET: now also J1.12; no longer J1.55
- net 3V3: now also C10.1, C11.1, R17.1, R19.1, U22.VDD, U23.VDD, U24.VDD, U27.3V3, U27.5V0, U27.VIO; no longer C19.1, C20.1, C21.1, U$2.3V3, U$2.5V0, U$2.VIO, U22.VDDIO, U22.VLDO, U23.VDDIO, U24.VDDIO, U3.4
- net 3V3_DISCO: now also C12.1, C19.1, U3.4; no longer C22.1
- net 5V0: now also C14.1, C20.1; no longer C7.1, C8.1
- net ADC2_PV1: no longer R11.1, R12.2, U21.3
- net ADC2_PV2: no longer R13.1, R14.2, U21.5
- net AF_CS: now also J2.62; no longer J2.56
- net FMC_A0: now also U27.AC1; no longer U$2.AC1
- net FMC_D0: now also U27.AD0; no longer U$2.AD0
- net FMC_D1: now also U27.AD1; no longer U$2.AD1
- net FMC_D2: now also U27.AD2; no longer U$2.AD2
- net FMC_D3: now also U27.AD3; no longer U$2.AD3
- net FMC_D4: now also U27.AD4; no longer U$2.AD4
- net FMC_D5: now also U27.AD5; no longer U$2.AD5
- net FMC_D6: now also U27.AD6; no longer U$2.AD6
- net FMC_D7: now also U27.AD7; no longer U$2.AD7
- net FMC_NE2: now also U27.AC0; no longer U$2.AC0
- net FMC_NOE: now also U27.AC2; no longer U$2.AC2
- net FMC_NWE: now also U27.AC3; no longer U$2.AC3
- net GND: now also C10.2, C11.2, C12.2, C16.2, U22.CHA, U23.CHA, U24.CHA, U27.GND-0, U27.GND-1, U27.SLD; no longer C21.2, C6.2, C7.2, C8.2, U$2.GND-0, U$2.GND-1, U$2.SLD, U22.GND, U23.GND, U24.GND
- net N$1: now also C15.1, C6.1; no longer C10.1, C11.1
- net N$22: now also C15.2, C6.2; no longer C10.2, C11.2
- net N$25: now also U27.PU2, U27.USB; no longer U$2.PU2, U$2.USB
- net N$3: now also C22.1; no longer C14.1
- net N$31: now also C8.2; no longer C16.2
- net N$38: now also C7.2; no longer C12.2
- net N$39: now also C21.2; no longer C15.2
- net N$40: now also C7.1; no longer C12.1
- net OF_CS: now also J1.35; no longer J2.62
- net PV1: now also R15.1, R16.1; no longer U23.VLDO
- net PV2: now also R10.1, R18.1; no longer U24.VLDO
- net SD_CS: now also J1.55; no longer J2.53
- net SPI5_MCLK: now also U22.GND, U23.GND, U24.GND; no longer U22.MCLK, U23.MCLK, U24.MCLK
- net VAF: now also C8.1; no longer C16.1
- net VSD: now also C16.1; no longer C6.1
- net VTH: now also C21.1; no longer C15.1
Routing:
- net !PLR_CLR: track 37.0 -> 228.7 mm, vias 0 -> 5
- net I2C3_SCL: track 102.5 -> 257.5 mm, vias 2 -> 5
- net I2C3_SDA: track 115.3 -> 253.5 mm, vias 2 -> 5
- net LD4: track 0.00 -> 107.0 mm, vias 0 -> 2
- net LD3: track 0.00 -> 97.2 mm, vias 0 -> 2
- net 3V3_DISCO: track 26.5 -> 117.9 mm, vias 0 -> 3
- net OF_CS: track 110.4 -> 25.9 mm
- net ADC3_PIO0: track 14.4 -> 95.4 mm, vias 1 -> 2
- net SPI5_MISO: track 173.5 -> 249.2 mm, vias 7 -> 10
- net ADC2_PV1: track 62.7 -> 132.3 mm, vias 1 -> 3
- net SPI5_MOSI: track 255.7 -> 325.2 mm, vias 9 -> 13
- net !USB_RST: track 16.3 -> 85.4 mm, vias 0 -> 2
- net ADC2_PV2: track 57.0 -> 125.1 mm, vias 0 -> 3
- net ADC2_PV0: track 46.5 -> 114.3 mm, vias 0 -> 3
- net SD_CS: track 75.0 -> 18.8 mm, vias 1 -> 0
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Other:
- board size 149.9 x 99.1 mm -> 149.9 x 120.7 mm
- board text added: "3V3"
- board text added: "5V0"
- board text added: "GND"
- board text added: "I2C3_SCL"
- board text added: "I2C3_SDA"
- board text added: "LAB-DEB429A - REV0"
- board text added: "LD3"
- board text added: "LD4"
- board text added: "PV1"
- board text added: "PV2"
- board text added: "SPI5_MCLK"
- board text added: "SPI5_MISO"
- board text added: "SPI5_MOSI"
