File: Hardware/LAB-DEB429A/cad/LAB-DEB429.brd (EAGLE design)
At the start: 149.9 x 120.7 mm, 102 parts, among them J1 TSW-132-02-S-D, J2 TSW-132-02-S-D, U1 LAB-ADSM300F, U10 SF-MICROSD, U11 25MPX, U12 LAB-PPS330D, U13 LAB-PPS330D, U14 LAB-PPS330D, U15 SI1143, U16 LAB-PPS330D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

Commit message: 1) Synchronizing some of the reference designators on the BOM vs the schematic (capacitors specifically) 2) Removing the 50pos connector from the BOM -- its supposed to be 64 ... dumbass.
Parts:
- R5, R6: value 2.2K -> 1K
Other:
- board text added: "LAB-DEB429A-REV1"
- board text removed: "LAB-DEB429A - REV1"
Changed lines of the file:
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@@
 <?xml version="1.0" encoding="utf-8"?>
 <!DOCTYPE eagle SYSTEM "eagle.dtd">
-<eagle version="7.3.0">
+<eagle version="6.6.0">
 <drawing>
 <settings>
@@
 <wire x1="8.255" y1="112.395" x2="8.255" y2="120.015" width="0.254" layer="25"/>
 <wire x1="8.255" y1="120.015" x2="48.895" y2="120.015" width="0.254" layer="25"/>
-<text x="85.725" y="1.905" size="3.81" layer="25">LAB-DEB429A - REV1</text>
+<text x="85.725" y="1.905" size="3.81" layer="25" font="vector">LAB-DEB429A-REV1</text>
 </plain>
 <attributes>
@@
 <pass name="Default">
 <param name="RoutingGrid" value="50mil"/>
-<param name="AutoGrid" value="1"/>
-<param name="Efforts" value="0"/>
-<param name="TopRouterVariant" value="1"/>
 <param name="tpViaShape" value="round"/>
 <param name="PrefDir.1" value="|"/>
@@
 <attribute name="VALUE" x="7.62" y="5.000625" size="1.27" layer="27" rot="R270"/>
 </element>
-<element name="R5" library="rcl" package="R0603" value="2.2K" x="80.645" y="112.7125" smashed="yes" rot="R270">
+<element name="R5" library="rcl" package="R0603" value="1K" x="80.645" y="112.7125" smashed="yes" rot="R270">
 <attribute name="NAME" x="85.09" y="113.665" size="1.016" layer="25" rot="R270"/>
 <attribute name="VALUE" x="78.74" y="113.3475" size="1.27" layer="27" rot="R270"/>
 </element>
-<element name="R6" library="rcl" package="R0603" value="2.2K" x="82.70875" y="112.7125" smashed="yes" rot="R90">
+<element name="R6" library="rcl" package="R0603" value="1K" x="82.70875" y="112.7125" smashed="yes" rot="R90">
 <attribute name="NAME" x="86.995" y="113.665" size="1.016" layer="25" rot="R270"/>
 <attribute name="VALUE" x="84.61375" y="112.0775" size="1.27" layer="27" rot="R90"/>
