File: Hardware/LAB-DEB429A/cad/LAB-DEB429.sch (EAGLE design)
At the start: 96 parts, among them J1 TSW-132-02-S-D, U1 LAB-ADSM300F, U10 SF-MICROSD, U11 25AA512, U12 LAB-PPS330D, U13 LAB-PPS330D, U14 LAB-PPS330D, U15 SI1143, U16 LAB-PPS330D, U17 25AA512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

Commit message: 1) Releasing first revision to MFG
Parts:
- added R10, R15, R16, R17, R18, R19: (no value), rcl:R-US_0204/7
- C10, C6, C7, C8, C9: value 10u -> 0.1u
- C14: value 47u -> 10u
- C15: value 0.22u -> 10u
- C16, C19, C20: value 0.1u -> 10u
- C21: value 0.1u -> 0.22u
- C22: value 0.1u -> 47u
- U11: value 25AA512 -> 25MPX; device PEGMA:25AA512 -> PEGMA:25MPX
- U17: value 25AA512 -> SST26VF; device PEGMA:25AA512 -> LAB304:SST26VF
- renumbered U$1 to U26, U$2 to U27, X1 to U25, X2 to J2
Connections:
- net FMC_A24 renamed LD3
- net FMC_A25 renamed LD4
- net LCD_B1 renamed LCD_B4
- net LCD_B9 renamed LCD_B7
- net MCU_SWK renamed MCU_SWC
- removed net !PLR_LDAC: U22.!LDAC, U23.!LDAC, U24.!LDAC
- removed net BOOT1: J2-30.1
- removed net FMC_NE1: J1-35.1
- removed net PV_DCHRG: J1-12.1
- removed net USB_OTG_FS_ID: J2-50.1
- new net FMC_D14: J2-53.1
- new net FMC_D15: J2-56.1
- new net N$176: R17.2, U22.CHA
- new net N$177: R19.2, U22.CHB
- new net N$178: R16.2, U23.CHB
- new net N$179: R15.2, U23.CHA
- new net N$180: R10.2, U24.CHB
- new net N$181: R18.2, U24.CHA
- new net N$182: R13.1, R14.2, U21G2.+IN
- new net N$183: R11.1, R12.2, U21G1.+IN
- net !PLR_CLR: now also J2-50.1
- net !USB_RST: now also J2-30.1
- net !WF_RESET: now also J1-12.1; no longer J1-55.1
- net 3V3: now also C10.1, C11.1, R17.1, R19.1; no longer C19.1, C20.1, C21.1, U22.VLDO, U3G1.-V
- net 3V3_DISCO: now also C12.1, C19.1, U3G1.-V; no longer C22.1
- net 5V0: now also C14.1, C20.1; no longer C7.1, C8.1
- net ADC2_PV1: no longer R11.1, R12.2, U21G1.+IN
- net ADC2_PV2: no longer R13.1, R14.2, U21G2.+IN
- net AF_CS: now also J2-62.1; no longer J2-56.1
- net GND: now also C10.2, C11.2, C12.2, C16.2; no longer C21.2, C6.2, C7.2, C8.2
- net N$1: now also C15.1, C6.1; no longer C10.1, C11.1
- net N$22: now also C15.2, C6.2; no longer C10.2, C11.2
- net N$3: now also C22.1; no longer C14.1
- net N$31: now also C8.2; no longer C16.2
- net N$38: now also C7.2; no longer C12.2
- net N$39: now also C21.2; no longer C15.2
- net N$40: now also C7.1; no longer C12.1
- net OF_CS: now also J1-35.1; no longer J2-62.1
- net PV1: now also R15.1, R16.1; no longer U23.VLDO
- net PV2: now also R10.1, R18.1; no longer U24.VLDO
- net SD_CS: now also J1-55.1; no longer J2-53.1
- net VAF: now also C8.1; no longer C16.1
- net VSD: now also C16.1; no longer C6.1
- net VTH: now also C21.1; no longer C15.1
Other:
- note added: "(Green)"
- note added: "(Red)"
- note added: "-- The lights may flicker when aux devices in use"
- note added: "Cannot use ACP/RF E2P Connector (I2C+ACP_RST in use)"
- note added: "MCU must not drive chip selects when MCU-Peripheral voltage is different"
- note added: "May need to bridge SB19 on DISCO board to connect HSE"
- note added: "Remove the MEMS from the DISCO board: CS and INT1/2 Pins are used"
- note added: "Using LD3 and LD4 as AUX0_CS and AUX1_CS"
- note removed: "LD3 (Green)"
- note removed: "LD4 (Red)"
- note removed: "Remove the MEMS from the DISCO board"
- note removed: "unnec"
- moved on the sheet: C10, C11, C12, C14, C15, C16, C19, C20, C21, C22, C6, C7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
