File: Hardware/LAB-PLR5010D/cad/LAB-PLR5010D.sch (EAGLE design)
At the start: 8 parts, among them J2 22-23-2021, J3 22-23-2021, U1 DAC8562, U2 LT3080, U3 LT3080

Commit message: 1) Committing final Rev0 of the PLR5010
Parts:
- removed J3: 22-23-2021, My Library-adm:22-23-2021
- added C3, C4: 33nf, SparkFun-Capacitors:1NF/1000PF-50V-10%(0603)
- J2: value 22-23-2021 -> 1729021; device My Library-adm:22-23-2021 -> My Library-adm:1729021
Connections:
- net GND: now also C3.2, C4.2; no longer J3-1.S
- net N$2: now also C3.1
- net N$3: now also C4.1
- net VB: now also J2-3.S; no longer J3-2.S
Other:
- moved on the sheet: J2-2
Changed lines of the file:
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@@
 <?xml version="1.0" encoding="utf-8"?>
 <!DOCTYPE eagle SYSTEM "eagle.dtd">
-<eagle version="6.5.0">
+<eagle version="6.6.0">
 <drawing>
 <settings>
@@
 <part name="SUPPLY1" library="SparkFun-Aesthetics" deviceset="3.3V" device=""/>
 <part name="GND" library="SparkFun-Aesthetics" deviceset="GND2" device="" value="gnd"/>
-<part name="J2" library="My Library-adm" deviceset="22-23-2021" device=""/>
-<part name="J3" library="My Library-adm" deviceset="22-23-2021" device=""/>
-<part name="GND1" library="SparkFun-Aesthetics" deviceset="GND2" device="" value="gnd"/>
 <part name="GND2" library="SparkFun-Aesthetics" deviceset="GND2" device="" value="gnd"/>
 <part name="J1" library="con-lstb" deviceset="MA10-1W" device=""/>
+<part name="J2" library="My Library-adm" deviceset="1729021" device=""/>
+<part name="C3" library="SparkFun-Capacitors" deviceset="1NF/1000PF-50V-10%(0603)" device="" value="33nf"/>
+<part name="C4" library="SparkFun-Capacitors" deviceset="1NF/1000PF-50V-10%(0603)" device="" value="33nf"/>
+<part name="GND1" library="SparkFun-Aesthetics" deviceset="GND2" device="" value="gnd"/>
+<part name="GND3" library="SparkFun-Aesthetics" deviceset="GND2" device="" value="gnd"/>
 </parts>
 <sheets>
@@
 <instance part="SUPPLY1" gate="G$1" x="96.52" y="121.92"/>
 <instance part="GND" gate="G$1" x="96.52" y="109.22" smashed="yes"/>
-<instance part="J2" gate="-1" x="259.08" y="157.48" smashed="yes">
-<attribute name="NAME" x="261.62" y="156.718" size="1.524" layer="95"/>
-<attribute name="VALUE" x="255.778" y="148.717" size="1.778" layer="96"/>
+<instance part="GND2" gate="G$1" x="256.54" y="121.92" smashed="yes"/>
+<instance part="J1" gate="1" x="33.02" y="114.3" rot="MR180"/>
+<instance part="J2" gate="-1" x="259.08" y="157.48"/>
+<instance part="J2" gate="-2" x="261.62" y="127"/>
+<instance part="J2" gate="-3" x="259.08" y="99.06"/>
+<instance part="C3" gate="G$1" x="177.8" y="111.76" smashed="yes" rot="MR270">
+<attribute name="NAME" x="174.244" y="116.459" size="1.778" layer="95" rot="MR180"/>
+<attribute name="VALUE" x="174.244" y="108.839" size="1.778" layer="96" rot="MR180"/>
 </instance>
-<instance part="J2" gate="-2" x="259.08" y="152.4"/>
-<instance part="J3" gate="-1" x="259.08" y="93.98" smashed="yes">
-<attribute name="NAME" x="261.62" y="93.218" size="1.524" layer="95"/>
-<attribute name="VALUE" x="255.778" y="90.297" size="1.778" layer="96"/>
+<instance part="C4" gate="G$1" x="177.8" y="99.06" smashed="yes" rot="MR270">
+<attribute name="NAME" x="174.244" y="103.759" size="1.778" layer="95" rot="MR180"/>
+<attribute name="VALUE" x="174.244" y="96.139" size="1.778" layer="96" rot="MR180"/>
 </instance>
-<instance part="J3" gate="-2" x="259.08" y="99.06" smashed="yes">
-<attribute name="NAME" x="261.62" y="98.298" size="1.524" layer="95"/>
-</instance>
-<instance part="GND1" gate="G$1" x="254" y="147.32" smashed="yes"/>
-<instance part="GND2" gate="G$1" x="254" y="88.9" smashed="yes"/>
-<instance part="J1" gate="1" x="33.02" y="114.3" rot="MR180"/>
+<instance part="GND1" gate="G$1" x="182.88" y="106.68" smashed="yes"/>
+<instance part="GND3" gate="G$1" x="182.88" y="93.98" smashed="yes"/>
 </instances>
 <busses>
@@
 <wire x1="172.72" y1="111.76" x2="172.72" y2="134.62" width="0.1524" layer="91"/>
 <pinref part="U1" gate="G$1" pin="VA"/>
+<pinref part="C3" gate="G$1" pin="1"/>
+<junction x="172.72" y="111.76"/>
 </segment>
 </net>
@@
 <pinref part="U1" gate="G$1" pin="VB"/>
 <wire x1="172.72" y1="99.06" x2="162.56" y2="99.06" width="0.1524" layer="91"/>
+<pinref part="C4" gate="G$1" pin="1"/>
+<junction x="172.72" y="99.06"/>
 </segment>
 </net>
@@
 </segment>
 <segment>
-<pinref part="J3" gate="-2" pin="S"/>
 <pinref part="U3" gate="G$1" pin="OUT"/>
 <wire x1="256.54" y1="99.06" x2="243.84" y2="99.06" width="0.1524" layer="91"/>
 <label x="256.54" y="99.06" size="1.778" layer="95" rot="MR0"/>
+<pinref part="J2" gate="-3" pin="S"/>
 </segment>
 </net>
@@
 </segment>
 <segment>
-<pinref part="J2" gate="-2" pin="S"/>
-<pinref part="GND1" gate="G$1" pin="3.3V"/>
-<wire x1="256.54" y1="152.4" x2="254" y2="152.4" width="0.1524" layer="91"/>
-<wire x1="254" y1="152.4" x2="254" y2="149.86" width="0.1524" layer="91"/>
-</segment>
-<segment>
-<pinref part="GND2" gate="G$1" pin="3.3V"/>
-<wire x1="254" y1="93.98" x2="254" y2="91.44" width="0.1524" layer="91"/>
-<pinref part="J3" gate="-1" pin="S"/>
-<wire x1="256.54" y1="93.98" x2="254" y2="93.98" width="0.1524" layer="91"/>
-</segment>
-<segment>
 <wire x1="40.64" y1="114.3" x2="53.34" y2="114.3" width="0.1524" layer="91"/>
 <pinref part="J1" gate="1" pin="5"/>
 <label x="53.34" y="114.3" size="1.778" layer="95" rot="MR0"/>
 </segment>
-</net>
+<segment>
+<pinref part="J2" gate="-2" pin="S"/>
+<pinref part="GND2" gate="G$1" pin="3.3V"/>
+<wire x1="256.54" y1="124.46" x2="256.54" y2="127" width="0.1524" layer="91"/>
+<wire x1="256.54" y1="127" x2="259.08" y2="127" width="0.1524" layer="91"/>
+</segment>
+<segment>
+<pinref part="C4" gate="G$1" pin="2"/>
+<wire x1="180.34" y1="99.06" x2="182.88" y2="99.06" width="0.1524" layer="91"/>
+<wire x1="182.88" y1="99.06" x2="182.88" y2="96.52" width="0.1524" layer="91"/>
+<pinref part="GND3" gate="G$1" pin="3.3V"/>
+</segment>
+<segment>
+<pinref part="C3" gate="G$1" pin="2"/>
+<wire x1="180.34" y1="111.76" x2="182.88" y2="111.76" width="0.1524" layer="91"/>
+<wire x1="182.88" y1="111.76" x2="182.88" y2="109.22" width="0.1524" layer="91"/>
+<pinref part="GND1" gate="G$1" pin="3.3V"/>
+</segment>
+</net>

Commit message: 1) Checkpoint before cleanup, final BOM and MFG
Parts:
- removed U2, U3: LT3080, LAB-PLR1010:LT3080
- added Q1, Q2: FZT849, LAB304:FZT849
- added R1, R2: (no value), rcl:R-US_R0603
- J1: device con-lstb:MA10-1W -> con-lstb:MA04-1
- J2: value 1729021 -> (none); device My Library-adm:1729021 -> con-lstb:MA04-1
Connections:
- removed net N$2: C3.1, U1.VA, U2.SET
- removed net VA: J1.1, J2-1.S, U2.OUT
- removed net VB: J1.10, J2-3.S, U3.OUT
- new net N$1: C3.1, R1.1, U1.VA
- new net N$4: Q1.B, R1.2
- new net N$5: Q2.B, R2.2
- net !CLR: now also J1.2; no longer J1.3
- net !CS: now also J1.3; no longer J1.7
- net !LDAC: now also J1.1; no longer J1.2
- net GND: now also J2.1, Q1.E, Q2.E; no longer J1.5, J2-2.S
- net MCLK: now also J1.4; no longer J1.8
- net MOSI: now also J2.2; no longer J1.9
- net N$3: now also R2.1; no longer U3.SET
- net VDDIO: now also J2.3; no longer J1.6, U2.VCNTRL, U3.VCNTRL
- net VDDLDO: now also J2.4, Q1.C, Q2.C; no longer J1.4, U2.IN, U3.IN
Other:
- moved on the sheet: C3, C4

Commit message: 1) Releasing new revision for MFG
Parts:
- R1, R2: value (none) -> 390R
- U1: device LAB-PLR1010:DAC8562 -> LAB-PLR5010D:DAC8562
Connections:
- removed net !LDAC: J1.1, U1.!LDAC
- removed net VDDIO: C1.1, C2.1, J2.3, U1.AVDD
- removed net VDDLDO: J2.4, Q1.C, Q2.C, U1.REFIN/OUT
- new net CHA: J2.1, Q1.C
- new net CHB: J2.4, Q2.C
- new net VDD: C1.1, C2.1, J2.3, U1.AVDD, U1.REFIN/OUT
- net GND: now also J1.1, U1.!LDAC; no longer J2.1

Commit message: 1) Updating the BOMs to include pricing and unifying passive MFG sources (samsung resistors).
Parts:
- C3, C4: value 33nf -> 0.01uF
Changed lines of the file:
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@@
 <?xml version="1.0" encoding="utf-8"?>
 <!DOCTYPE eagle SYSTEM "eagle.dtd">
-<eagle version="6.6.0">
+<eagle version="7.3.0">
 <drawing>
 <settings>
@@
 <part name="SUPPLY1" library="SparkFun-Aesthetics" deviceset="3.3V" device=""/>
 <part name="GND" library="SparkFun-Aesthetics" deviceset="GND2" device="" value="gnd"/>
-<part name="C3" library="SparkFun-Capacitors" deviceset="1NF/1000PF-50V-10%(0603)" device="" value="33nf"/>
-<part name="C4" library="SparkFun-Capacitors" deviceset="1NF/1000PF-50V-10%(0603)" device="" value="33nf"/>
+<part name="C3" library="SparkFun-Capacitors" deviceset="1NF/1000PF-50V-10%(0603)" device="" value="0.01uF"/>
+<part name="C4" library="SparkFun-Capacitors" deviceset="1NF/1000PF-50V-10%(0603)" device="" value="0.01uF"/>
 <part name="GND1" library="SparkFun-Aesthetics" deviceset="GND2" device="" value="gnd"/>
 <part name="GND3" library="SparkFun-Aesthetics" deviceset="GND2" device="" value="gnd"/>

Commit message: 1) Updating the PLR-5010D as-built 2) Adding the linearization xls
Parts:
- added R3, R4: 27K, rcl:R-US_R0603
- R1, R2: value 390R -> 3.9K
Connections:
- net CHA: now also R3.2
- net CHB: now also R4.2
- net N$4: now also R3.1
- net N$5: now also R4.1
Other:
- moved on the sheet: J1, J2
Changed lines of the file:
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@@
 <?xml version="1.0" encoding="utf-8"?>
 <!DOCTYPE eagle SYSTEM "eagle.dtd">
-<eagle version="7.3.0">
+<eagle version="6.6.0">
 <drawing>
 <settings>
@@
 <part name="GND4" library="SparkFun-Aesthetics" deviceset="GND2" device="" value="gnd"/>
 <part name="GND5" library="SparkFun-Aesthetics" deviceset="GND2" device="" value="gnd"/>
-<part name="R1" library="rcl" deviceset="R-US_" device="R0603" value="390R"/>
-<part name="R2" library="rcl" deviceset="R-US_" device="R0603" value="390R"/>
+<part name="R1" library="rcl" deviceset="R-US_" device="R0603" value="3.9K"/>
+<part name="R2" library="rcl" deviceset="R-US_" device="R0603" value="3.9K"/>
 <part name="J1" library="con-lstb" deviceset="MA04-1" device=""/>
 <part name="J2" library="con-lstb" deviceset="MA04-1" device=""/>
 <part name="U1" library="LAB-PLR5010D" deviceset="DAC8562" device=""/>
+<part name="R3" library="rcl" deviceset="R-US_" device="R0603" value="27K"/>
+<part name="R4" library="rcl" deviceset="R-US_" device="R0603" value="27K"/>
 </parts>
 <sheets>
@@
 <instance part="R1" gate="G$1" x="185.42" y="111.76"/>
 <instance part="R2" gate="G$1" x="185.42" y="99.06"/>
-<instance part="J1" gate="1" x="68.58" y="86.36"/>
-<instance part="J2" gate="1" x="68.58" y="68.58"/>
+<instance part="J1" gate="1" x="60.96" y="114.3"/>
+<instance part="J2" gate="1" x="60.96" y="96.52"/>
 <instance part="U1" gate="G$1" x="139.7" y="106.68"/>
+<instance part="R3" gate="G$1" x="198.12" y="116.84" smashed="yes" rot="MR90">
+<attribute name="NAME" x="196.85" y="115.7986" size="1.778" layer="95" rot="MR0"/>
+<attribute name="VALUE" x="196.85" y="113.538" size="1.778" layer="96" rot="MR0"/>
+</instance>
+<instance part="R4" gate="G$1" x="218.44" y="104.14" smashed="yes" rot="MR90">
+<attribute name="NAME" x="217.17" y="103.0986" size="1.778" layer="95" rot="MR0"/>
+<attribute name="VALUE" x="217.17" y="100.838" size="1.778" layer="96" rot="MR0"/>
+</instance>
 </instances>
 <busses>
@@
 </segment>
 <segment>
-<wire x1="76.2" y1="88.9" x2="88.9" y2="88.9" width="0.1524" layer="91"/>
+<wire x1="68.58" y1="116.84" x2="81.28" y2="116.84" width="0.1524" layer="91"/>
 <pinref part="J1" gate="1" pin="4"/>
-<label x="88.9" y="88.9" size="1.778" layer="95" rot="MR0"/>
+<label x="81.28" y="116.84" size="1.778" layer="95" rot="MR0"/>
 </segment>
 </net>
@@
 </segment>
 <segment>
-<wire x1="76.2" y1="86.36" x2="88.9" y2="86.36" width="0.1524" layer="91"/>
+<wire x1="68.58" y1="114.3" x2="81.28" y2="114.3" width="0.1524" layer="91"/>
 <pinref part="J1" gate="1" pin="3"/>
-<label x="88.9" y="86.36" size="1.778" layer="95" rot="MR0"/>
+<label x="81.28" y="114.3" size="1.778" layer="95" rot="MR0"/>
 </segment>
 </net>
@@
 </segment>
 <segment>
-<wire x1="76.2" y1="66.04" x2="88.9" y2="66.04" width="0.1524" layer="91"/>
-<label x="88.9" y="66.04" size="1.778" layer="95" rot="MR0"/>
+<wire x1="68.58" y1="93.98" x2="81.28" y2="93.98" width="0.1524" layer="91"/>
+<label x="81.28" y="93.98" size="1.778" layer="95" rot="MR0"/>
 <pinref part="J2" gate="1" pin="2"/>
 </segment>
@@
 </segment>
 <segment>
-<wire x1="76.2" y1="81.28" x2="88.9" y2="81.28" width="0.1524" layer="91"/>
+<wire x1="68.58" y1="109.22" x2="81.28" y2="109.22" width="0.1524" layer="91"/>
 <pinref part="J1" gate="1" pin="1"/>
-<label x="88.9" y="81.28" size="1.778" layer="95" rot="MR0"/>
+<label x="81.28" y="109.22" size="1.778" layer="95" rot="MR0"/>
 </segment>
 </net>
@@
 </segment>
 <segment>
-<wire x1="88.9" y1="83.82" x2="76.2" y2="83.82" width="0.1524" layer="91"/>
+<wire x1="81.28" y1="111.76" x2="68.58" y2="111.76" width="0.1524" layer="91"/>
 <pinref part="J1" gate="1" pin="2"/>
-<label x="88.9" y="83.82" size="1.778" layer="95" rot="MR0"/>
+<label x="81.28" y="111.76" size="1.778" layer="95" rot="MR0"/>
 </segment>
 </net>
@@
 <pinref part="R1" gate="G$1" pin="2"/>
 <pinref part="Q1" gate="G$1" pin="B"/>
-<wire x1="190.5" y1="111.76" x2="198.12" y2="111.76" width="0.1524" layer="91"/>
+<pinref part="R3" gate="G$1" pin="1"/>
+<junction x="198.12" y="111.76"/>
+<wire x1="198.12" y1="111.76" x2="190.5" y2="111.76" width="0.1524" layer="91"/>
 </segment>
 </net>
@@
 <pinref part="Q2" gate="G$1" pin="B"/>
 <wire x1="190.5" y1="99.06" x2="218.44" y2="99.06" width="0.1524" layer="91"/>
+<pinref part="R4" gate="G$1" pin="1"/>
+<junction x="218.44" y="99.06"/>
 </segment>
 </net>
@@
 <segment>
 <pinref part="Q1" gate="G$1" pin="C"/>
-<wire x1="203.2" y1="116.84" x2="203.2" y2="124.46" width="0.1524" layer="91"/>
+<wire x1="203.2" y1="116.84" x2="203.2" y2="121.92" width="0.1524" layer="91"/>
 <label x="203.2" y="124.46" size="1.778" layer="95"/>
-</segment>
-<segment>
-<wire x1="88.9" y1="63.5" x2="76.2" y2="63.5" width="0.1524" layer="91"/>
+<pinref part="R3" gate="G$1" pin="2"/>
+<wire x1="203.2" y1="121.92" x2="203.2" y2="124.46" width="0.1524" layer="91"/>
+<wire x1="198.12" y1="121.92" x2="203.2" y2="121.92" width="0.1524" layer="91"/>
+<junction x="203.2" y="121.92"/>
+</segment>
+<segment>
+<wire x1="81.28" y1="91.44" x2="68.58" y2="91.44" width="0.1524" layer="91"/>
 <pinref part="J2" gate="1" pin="1"/>
-<label x="88.9" y="63.5" size="1.778" layer="95" rot="MR0"/>
+<label x="81.28" y="91.44" size="1.778" layer="95" rot="MR0"/>
 </segment>
 </net>
@@
 <segment>
 <pinref part="Q2" gate="G$1" pin="C"/>
-<wire x1="223.52" y1="104.14" x2="223.52" y2="124.46" width="0.1524" layer="91"/>
+<wire x1="223.52" y1="104.14" x2="223.52" y2="109.22" width="0.1524" layer="91"/>
 <label x="223.52" y="124.46" size="1.778" layer="95"/>
-</segment>
-<segment>
-<wire x1="76.2" y1="71.12" x2="88.9" y2="71.12" width="0.1524" layer="91"/>
+<pinref part="R4" gate="G$1" pin="2"/>
+<wire x1="223.52" y1="109.22" x2="223.52" y2="124.46" width="0.1524" layer="91"/>
+<wire x1="218.44" y1="109.22" x2="223.52" y2="109.22" width="0.1524" layer="91"/>
+<junction x="223.52" y="109.22"/>
+</segment>
+<segment>
+<wire x1="68.58" y1="99.06" x2="81.28" y2="99.06" width="0.1524" layer="91"/>
 <pinref part="J2" gate="1" pin="4"/>
-<label x="88.9" y="71.12" size="1.778" layer="95" rot="MR0"/>
+<label x="81.28" y="99.06" size="1.778" layer="95" rot="MR0"/>
 </segment>
 </net>
 <net name="VDD" class="0">
 <segment>
-<wire x1="76.2" y1="68.58" x2="88.9" y2="68.58" width="0.1524" layer="91"/>
+<wire x1="68.58" y1="96.52" x2="81.28" y2="96.52" width="0.1524" layer="91"/>
 <pinref part="J2" gate="1" pin="3"/>
-<label x="88.9" y="68.58" size="1.778" layer="95" rot="MR0"/>
-</segment>
-<segment>
+<label x="81.28" y="96.52" size="1.778" layer="95" rot="MR0"/>
+</segment>
+<segment>
